Commit message: feat: update puzzlebot simulation and navigation config

File: puzzlebot_description/urdf/base.xacro (robot description, xacro)
@@ -6,5 +6,5 @@
       <origin xyz="0 0 0" rpy="0 0 0"/>
       <geometry>
-        <mesh filename="package://puzzlebot_description/meshes/Puzzlebot_Jetson_Lidar_Edition_Base.stl"/>
+        <mesh filename="package://puzzlebot_description/meshes/Puzzlebot_Jetson_Lidar_Edition_Base.stl" scale="${mesh_scale} ${mesh_scale} ${mesh_scale}"/>
       </geometry>
       <material name="yellow">
@@ -23,5 +23,6 @@
     <parent link="base_footprint"/>
     <child  link="base_link"/>
-    <origin xyz="0 0 0.05" rpy="0 0 0"/>
+    <!-- 0.0368 = wheel_radius (0.035) + wheel offset (0.00175) -->
+    <origin xyz="0 0 0.0368" rpy="0 0 0"/>
   </joint>
 </robot>

File: puzzlebot_description/urdf/gazebo_plugins.xacro (robot description, xacro)
@@ -6,15 +6,15 @@
   <gazebo reference="wheel_r_link">
     <material>Gazebo/DarkGrey</material>
-    <mu1>1.0</mu1>
-    <mu2>1.0</mu2>
-    <kp>500000.0</kp>
-    <kd>10.0</kd>
+    <mu1>0.8</mu1>
+    <mu2>0.5</mu2>
+    <kp>1000000.0</kp>
+    <kd>100.0</kd>
   </gazebo>
   <gazebo reference="wheel_l_link">
     <material>Gazebo/DarkGrey</material>
-    <mu1>1.0</mu1>
-    <mu2>1.0</mu2>
-    <kp>500000.0</kp>
-    <kd>10.0</kd>
+    <mu1>0.8</mu1>
+    <mu2>0.5</mu2>
+    <kp>1000000.0</kp>
+    <kd>100.0</kd>
   </gazebo>
   <gazebo reference="caster_link">
@@ -33,11 +33,11 @@
       <wheel_separation>${wheel_separation}</wheel_separation>
       <wheel_diameter>${2*wheel_radius}</wheel_diameter>
-      <max_wheel_torque>20</max_wheel_torque>
-      <max_wheel_acceleration>1.0</max_wheel_acceleration>
+      <max_wheel_torque>50</max_wheel_torque>
+      <max_wheel_acceleration>3.0</max_wheel_acceleration>
       <odometry_frame>odom</odometry_frame>
       <robot_base_frame>base_footprint</robot_base_frame>
       <publish_odom>true</publish_odom>
       <publish_odom_tf>true</publish_odom_tf>
-      <publish_wheel_tf>false</publish_wheel_tf>
+      <publish_wheel_tf>true</publish_wheel_tf>
       <ros>
         <remapping>cmd_vel:=cmd_vel</remapping>
@@ -62,5 +62,5 @@
         </scan>
         <range>
-          <min>0.12</min>
+          <min>0.08</min>
           <max>5.0</max>
           <resolution>0.015</resolution>

File: puzzlebot_description/urdf/puzzlebot.urdf.xacro (robot description, xacro)
@@ -2,19 +2,21 @@
 <robot name="puzzlebot" xmlns:xacro="http://www.ros.org/wiki/xacro">
   <!-- ============================================================
-       PROPERTIES — parametros fisicos del Puzzlebot
+       PROPERTIES — Puzzlebot escalado al 70% para caber en pasillos estrechos
+       Tamano efectivo: 12.6 x 10.5 cm (era 18 x 15 cm)
        ============================================================ -->
+  <xacro:property name="mesh_scale"      value="0.7"/>
   <xacro:property name="base_mass"       value="0.5"/>
   <xacro:property name="wheel_mass"      value="0.05"/>
   <xacro:property name="caster_mass"     value="0.02"/>
   <xacro:property name="lidar_mass"      value="0.17"/>
-  <xacro:property name="base_length"     value="0.18"/>
-  <xacro:property name="base_width"      value="0.15"/>
-  <xacro:property name="base_height"     value="0.07"/>
-  <xacro:property name="wheel_radius"    value="0.05"/>
-  <xacro:property name="wheel_width"     value="0.025"/>
-  <xacro:property name="wheel_separation" value="0.19"/>
-  <xacro:property name="caster_radius"   value="0.02"/>
-  <xacro:property name="lidar_radius"    value="0.035"/>
-  <xacro:property name="lidar_height"    value="0.04"/>
+  <xacro:property name="base_length"     value="0.126"/>
+  <xacro:property name="base_width"      value="0.105"/>
+  <xacro:property name="base_height"     value="0.05"/>
+  <xacro:property name="wheel_radius"    value="0.035"/>
+  <xacro:property name="wheel_width"     value="0.018"/>
+  <xacro:property name="wheel_separation" value="0.133"/>
+  <xacro:property name="caster_radius"   value="0.014"/>
+  <xacro:property name="lidar_radius"    value="0.025"/>
+  <xacro:property name="lidar_height"    value="0.03"/>
   <!-- ============================================================
        INCLUDES — modulos del robot

File: puzzlebot_description/urdf/wheels.xacro (robot description, xacro)
@@ -6,5 +6,5 @@
         <origin xyz="0 0 0" rpy="1.5708 0 0"/>
         <geometry>
-          <mesh filename="package://puzzlebot_description/meshes/Puzzlebot_Wheel.stl"/>
+          <mesh filename="package://puzzlebot_description/meshes/Puzzlebot_Wheel.stl" scale="${mesh_scale} ${mesh_scale} ${mesh_scale}"/>
         </geometry>
         <material name="dark_grey">
@@ -23,5 +23,5 @@
       <parent link="base_link"/>
       <child  link="${name}_link"/>
-      <origin xyz="0.052 ${y_reflect * wheel_separation/2.0} -0.0025" rpy="0 0 0"/>
+      <origin xyz="0.036 ${y_reflect * wheel_separation/2.0} -0.00175" rpy="0 0 0"/>
       <axis xyz="0 1 0"/>
       <dynamics damping="0.01" friction="0.1"/>
@@ -34,5 +34,5 @@
       <origin xyz="0 0 0" rpy="0 0 0"/>
       <geometry>
-        <mesh filename="package://puzzlebot_description/meshes/Puzzlebot_Caster_Wheel.stl"/>
+        <mesh filename="package://puzzlebot_description/meshes/Puzzlebot_Caster_Wheel.stl" scale="${mesh_scale} ${mesh_scale} ${mesh_scale}"/>
       </geometry>
       <material name="grey">
@@ -51,5 +51,5 @@
     <parent link="base_link"/>
     <child  link="caster_link"/>
-    <origin xyz="-0.095 0.0 -0.03" rpy="0 0 0"/>
+    <origin xyz="-0.067 0.0 -0.023" rpy="0 0 0"/>
   </joint>
 </robot>
